Commit message: Created IKFast translational 3D solver and implemented it in MoveIt

File: open_manipulator_description/urdf/open_manipulator.gazebo.urdf (robot description, URDF)
Before this commit: robot open_manipulator, 9 links, 8 joints
Links:
- added link link0
Joints:
- added joint joint0: type fixed, parent link0, child link1, origin xyz=0.0 0.0 0.0 rpy=0 0 0

File: open_manipulator_description/urdf/open_manipulator.urdf.xacro (robot description, xacro)
@@ -2,4 +2,12 @@
 <!-- Open_Manipulator Chain -->
 <robot xmlns:xacro="http://ros.org/wiki/xacro">
+  <!-- Base link (link 0) -->
+  <link name="link0"/>
+  <!-- Joint 0 -->
+  <joint name="joint0" type="fixed">
+    <parent link="link0"/>
+    <child link="link1"/>
+    <origin xyz="0.0 0.0 0.0" rpy="0 0 0"/>
+  </joint>
   <!-- Link 1 -->
   <link name="link1">
