Commit message: joint_group_position_controller and moveit_servo launch and config files

File: open_manipulator_description/urdf/open_manipulator.urdf.xacro (robot description, xacro)
@@ -3,8 +3,8 @@
 <robot xmlns:xacro="http://ros.org/wiki/xacro">
   <!-- Base link (link 0) -->
-  <link name="link0"/>
+  <link name="world"/>
   <!-- Joint 0 -->
   <joint name="joint0" type="fixed">
-    <parent link="link0"/>
+    <parent link="world"/>
     <child link="link1"/>
     <origin xyz="0.0 0.0 0.0" rpy="0 0 0"/>

File: open_manipulator_description/urdf/open_manipulator_gazebo.urdf (robot description, URDF)
Before this commit: robot open_manipulator, 10 links, 9 joints
Links:
- removed link link0
- added link world
Joints:
- joint joint0: parent link0 -> world
